File: mistance_PCB/mistance_PCB.kicad_sch (KiCad schematic)
At the start: 17 parts, among them J1 USB_B_Micro, Q1 Q_PMOS_DSG, U1 ESP32-WROOM-32E, U2 TPS61200DRC, U3 MCP73831-2-OT

Commit message: PCB update
Parts:
- C1, C2, C3, C4, C5: footprint (none) -> Capacitor_SMD:C_1210_3225Metric
- D1: footprint (none) -> Diode_SMD:DIOM5226X220N
- J1: footprint (none) -> Connector_USB:USB_Micro-B_Amphenol_10103594-0001LF_Horizontal
- Q1: footprint (none) -> SI2333DS-T1-E3:SOT95P237X112-3N
- R1, R2: footprint (none) -> Resistor_SMD:R_1210_3225Metric
- R3: footprint Resistor_SMD:R_0815_2038Metric -> Resistor_SMD:R_0603_1608Metric
- R4: footprint (none) -> Resistor_SMD:R_0603_1608Metric
Changed lines of the file:
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@@
 			)
 		)
-		(property "Footprint" ""
+		(property "Footprint" "Capacitor_SMD:C_1210_3225Metric"
 			(at 228.2952 69.85 0)
 			(effects
@@
 			)
 		)
-		(property "Footprint" ""
+		(property "Footprint" "Resistor_SMD:R_1210_3225Metric"
 			(at 170.942 54.61 90)
 			(effects
@@
 			)
 		)
-		(property "Footprint" ""
+		(property "Footprint" "Resistor_SMD:R_0603_1608Metric"
 			(at 144.272 29.21 90)
 			(effects
@@
 			)
 		)
-		(property "Footprint" ""
+		(property "Footprint" "Resistor_SMD:R_1210_3225Metric"
 			(at 170.942 64.77 90)
 			(effects
@@
 			)
 		)
-		(property "Footprint" ""
+		(property "Footprint" "Capacitor_SMD:C_1210_3225Metric"
 			(at 117.8052 46.99 0)
 			(effects
@@
 			)
 		)
-		(property "Footprint" ""
+		(property "Footprint" "Capacitor_SMD:C_1210_3225Metric"
 			(at 169.8752 68.58 0)
 			(effects
@@
 			)
 		)
-		(property "Footprint" "Resistor_SMD:R_0815_2038Metric"
+		(property "Footprint" "Resistor_SMD:R_0603_1608Metric"
 			(at 118.872 50.8 90)
 			(effects
@@
 			)
 		)
-		(property "Footprint" ""
+		(property "Footprint" "Capacitor_SMD:C_1210_3225Metric"
 			(at 218.1352 69.85 0)
 			(effects
@@
 			)
 		)
-		(property "Footprint" ""
+		(property "Footprint" "Connector_USB:USB_Micro-B_Amphenol_10103594-0001LF_Horizontal"
 			(at 107.95 43.18 0)
 			(effects
@@
 			)
 		)
-		(property "Footprint" ""
+		(property "Footprint" "Capacitor_SMD:C_1210_3225Metric"
 			(at 148.2852 50.8 0)
 			(effects
@@
 			)
 		)
-		(property "Footprint" ""
+		(property "Footprint" "SI2333DS-T1-E3:SOT95P237X112-3N"
 			(at 163.83 44.45 0)
 			(effects
@@
 			)
 		)
-		(property "Footprint" ""
+		(property "Footprint" "Diode_SMD:DIOM5226X220N"
 			(at 186.69 25.4 0)
 			(effects
