File: mistance_PCB/mistance_PCB.kicad_pcb (KiCad board)
At the start: 2 copper layers, 86.4 x 99.3 mm, 66 parts, among them J1 USB_B_Micro, J2 USB_B_Micro, J3 GRPB052VWVN-RC, J4 OLED, J5 SMA-J-P-X-ST-TH1, Q1 Q_PMOS_DSG, U1 ESP32-WROOM-32E, U2 TPS61200DRC, U3 MCP73831-2-OT, U4 AMS1117-3.3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

Commit message: PCB last add GND plain
Routing:
- net GND: track 419.7 -> 439.0 mm
- net USB 5V OUT: track 10.7 -> 11.2 mm
- net MOSI: track 52.2 -> 52.6 mm, vias 2 -> 4
- net I2C SCL: track 87.3 -> 87.7 mm, vias 0 -> 4
- net 3.3V OUT: vias 6 -> 8
Other:
- outline, holes or cut-outs redrawn
