File: mistance_PCB/mistance_PCB_host/mistance_PCB_host.kicad_sch (KiCad schematic)
At the start: 88 parts, among them J3 GRPB052VWVN-RC, J4 OLED, J5 SMA-J-P-X-ST-TH1, Q1 Q_PMOS_DSG, Q2 UMH3N, U1 ESP32-WROOM-32E, U2 TPS61200DRC, U3 MCP73831-2-OT, U4 AMS1117-3.3, U5 CP2104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

Commit message: host PCB and SCH bug fix
Parts:
- removed C25: 1uF, Capacitor_SMD:C_0603_1608Metric, symbol Device:C
- removed C26: 10uF, Capacitor_SMD:C_0603_1608Metric, symbol Device:C
- removed R5: 10K, Resistor_SMD:R_0603_1608Metric, symbol Device:R
- removed U6: TPS3839DBZ, Package_TO_SOT_SMD:SOT-23, symbol Power_Supervisor:TPS3839DBZ
- added C37: 1uF, Capacitor_SMD:C_0603_1608Metric, symbol Device:C
- added R30: 22R, Resistor_SMD:R_0402_1005Metric, symbol Device:R
- R9: value 100K -> 10K
Connections:
- net 3.3V OUT: now also C23.1, R9.2
- net EN: now also R9.1, U1.3 (EN), C37.1, R30.2; no longer C27.2, S1.3, S1.4
- net GND: now also C24.1, C37.2; no longer R9.2
- new net: C27.2, R30.1, S1.3, S1.4
- no-connect marks 31 -> 32
Other:
- moved on the sheet: C23, C27, S1

Commit message: modify
Parts:
- R16, R17, R18, R19, R20: value 100K -> 10K
Connections:
- no-connect marks 32 -> 31

Commit message: host code
Changed lines of the file:
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@@
 	)
 	(global_label "MISO"
-		(shape output)
+		(shape input)
 		(at 241.3 109.22 180)
 		(fields_autoplaced yes)
@@
 	)
 	(global_label "MISO"
-		(shape input)
+		(shape output)
 		(at 72.39 107.95 0)
 		(fields_autoplaced yes)

Commit message: host code modify & host PCB and SCH modify
Parts:
- added C25: 22uF, Capacitor_SMD:C_0805_2012Metric, symbol Device:C
- added C7: 1uF, Capacitor_SMD:C_0603_1608Metric, symbol Device:C
- added R31: 1K, Resistor_SMD:R_0603_1608Metric, symbol Device:R
- added R5: 100R, Resistor_SMD:R_0402_1005Metric, symbol Device:R
- added U6: L86-M33, L86-M33:XCVR_L86-M33, symbol L86-M33:L86-M33
Connections:
- net 3.3V OUT: now also C25.1, C7.1, U6.4 (VCC), U6.5 (V_BCKP)
- net GND: now also C25.2, C7.2, R31.1, U6.12 (GND), U6.3 (GND)
- net GPS_Reset: now reaches U1.26 (IO4)
- net GPS_Reset: now also R5.1
- net GPS_TX: now reaches U1.8 (IO32)
- net GPS_TX: now also U6.2 (TXD1)
- net GPS_Rx: now reaches U1.9 (IO33)
- net GPS_Rx: now also U6.1 (RXD1)
- new net: R31.2, R5.2, U6.10 (~{RESET})
- no-connect marks 31 -> 32
Other:
- moved on the sheet: C13, C14, C15, C18, C19, C27, C35, C37, C6, C8, J3, J4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

Commit message: PCB and code modify
Connections:
- net 5v OUT: now also FL1.2, UART1.A4 (VBUS), UART1.A9 (VBUS), UART1.B4 (VBUS), UART1.B9 (VBUS)
Changed lines of the file:
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@@
 	)
 	(junction
+		(at 204.47 152.4)
+		(diameter 0)
+		(color 0 0 0 0)
+	)
+	(junction
 		(at 203.2 118.11)
 		(diameter 0)
@@
 	(wire
 		(pts
-			(xy 204.47 135.89) (xy 204.47 158.75)
+			(xy 204.47 135.89) (xy 204.47 152.4)
 		)
 		(stroke
@@
 	(wire
 		(pts
+			(xy 204.47 152.4) (xy 205.74 152.4)
+		)
+		(stroke
+			(width 0)
+			(type default)
+		)
+	)
+	(wire
+		(pts
 			(xy 147.32 50.8) (xy 147.32 52.07)
 		)
@@
 	(wire
 		(pts
+			(xy 204.47 152.4) (xy 204.47 158.75)
+		)
+		(stroke
+			(width 0)
+			(type default)
+		)
+	)
+	(wire
+		(pts
 			(xy 247.65 81.28) (xy 250.19 81.28)
 		)
@@
 	(wire
 		(pts
-			(xy 82.55 95.25) (xy 82.55 104.14)
+			(xy 82.55 95.25) (xy 82.55 99.06)
 		)
 		(stroke
@@
 		)
 	)
+	(global_label "5v OUT"
+		(shape input)
+		(at 205.74 152.4 0)
+		(fields_autoplaced yes)
+		(effects
+			(font
+				(size 1.27 1.27)
+			)
+			(justify left)
+		)
+		(property "Intersheetrefs" "${INTERSHEET_REFS}"
+			(at 215.4985 152.4 0)
+			(effects
+				(font
+					(size 1.27 1.27)
+				)
+				(justify left)
+				(hide yes)
+			)
+		)
+	)
 	(global_label "3.3V OUT"
 		(shape output)
@@
 	(symbol
 		(lib_id "power:GND")
-		(at 82.55 104.14 0)
+		(at 82.55 99.06 0)
 		(unit 1)
 		(exclude_from_sim no)
@@
 		(fields_autoplaced yes)
 		(property "Reference" "#PWR08"
-			(at 82.55 110.49 0)
+			(at 82.55 105.41 0)
 			(effects
 				(font
@@
 		)
 		(property "Value" "GND"
-			(at 82.55 109.22 0)
+			(at 82.55 104.14 0)
 			(effects
 				(font
@@
 		)
 		(property "Footprint" ""
-			(at 82.55 104.14 0)
+			(at 82.55 99.06 0)
 			(effects
 				(font
@@
 		)
 		(property "Datasheet" ""
-			(at 82.55 104.14 0)
+			(at 82.55 99.06 0)
 			(effects
 				(font
@@
 		)
 		(property "Description" "Power symbol creates a global label with name \"GND\" , ground"
-			(at 82.55 104.14 0)
+			(at 82.55 99.06 0)
 			(effects
 				(font
