File: mistance_PCB/FLP_PCB_host/FLP_PCB_host.kicad_pcb (KiCad board)
At the start: 2 copper layers, 90 x 90.5 mm, 91 parts, among them J3 GRPB052VWVN-RC, J4 OLED, J5 SMA-J-P-X-ST-TH1, Q1 Q_PMOS_DSG, Q2 UMH3N, U1 ESP32-WROOM-32E, U2 TPS61200DRC, U3 MCP73831-2-OT, U4 AMS1117-3.3, U5 CP2104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

Commit message: name fix and grb file add
Parts:
- Ctrl1: value Ctrl -> SKRPABE010
- D1: value D_Schottky -> MBRA160T3G
- Down1: value Down -> SKRPABE010
- Enter&space1: value Enter&space -> SKRPABE010
- Find_Host1: value Find_Host -> SKRPABE010
- L4: value WE-TPC_2811 -> 744028000056
- UART1: value USB_C_Receptacle_USB2.0_16P -> 12402012E212A
- Up1: value Up -> SKRPABE010
- Y1: value Crystal -> 32MHz
- moved R5 0.43 mm to (64.2, 68.5)
- moved R24 0.10 mm to (29.4, 59.0)
Routing:
- net GND: track 478.4 -> 482.1 mm
