File: mistance_PCB/FLP_PCB_host/FLP_PCB_host.kicad_sch (KiCad schematic)
At the start: 91 parts, among them J3 GRPB052VWVN-RC, J4 OLED, J5 SMA-J-P-X-ST-TH1, Q1 Q_PMOS_DSG, Q2 UMH3N, U1 ESP32-WROOM-32E, U2 TPS61200DRC, U3 MCP73831-2-OT, U4 AMS1117-3.3, U5 CP2104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

Commit message: name fix and grb file add
Parts:
- Charger1: value Charger -> 10103594-0001LF
- Ctrl1: value Ctrl -> SKRPABE010
- D1: value D_Schottky -> MBRA160T3G
- Down1: value Down -> SKRPABE010
- Enter&space1: value Enter&space -> SKRPABE010
- Find_Host1: value Find_Host -> SKRPABE010
- L4: value WE-TPC_2811 -> 744028000056
- UART1: value USB_C_Receptacle_USB2.0_16P -> 12402012E212A
- Up1: value Up -> SKRPABE010
- Y1: value Crystal -> 32MHz
Changed lines of the file:
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@@
 			)
 		)
-		(property "Value" "Ctrl"
+		(property "Value" "SKRPABE010"
 			(at 242.57 161.29 0)
 			(effects
@@
 			)
 		)
-		(property "Value" "WE-TPC_2811"
+		(property "Value" "744028000056"
 			(at 259.08 8.89 0)
 			(effects
@@
 			)
 		)
-		(property "Value" "Down"
+		(property "Value" "SKRPABE010"
 			(at 242.57 154.94 0)
 			(effects
@@
 			)
 		)
-		(property "Value" "USB_C_Receptacle_USB2.0_16P"
+		(property "Value" "12402012E212A"
 			(at 231.14 121.9199 0)
 			(effects
@@
 			)
 		)
-		(property "Value" "Enter&space"
+		(property "Value" "SKRPABE010"
 			(at 242.57 142.24 0)
 			(effects
@@
 			)
 		)
-		(property "Value" "Up"
+		(property "Value" "SKRPABE010"
 			(at 242.57 147.32 0)
 			(effects
@@
 			)
 		)
-		(property "Value" "Charger"
+		(property "Value" "10103594-0001LF"
 			(at 104.14 31.75 0)
 			(effects
@@
 			)
 		)
-		(property "Value" "Crystal"
+		(property "Value" "32MHz"
 			(at 241.3 76.1999 90)
 			(effects
@@
 			)
 		)
-		(property "Value" "Find_Host"
+		(property "Value" "SKRPABE010"
 			(at 242.57 135.89 0)
 			(effects
@@
 		(on_board yes)
 		(dnp no)
-		(fields_autoplaced yes)
 		(property "Reference" "C15"
 			(at 59.69 179.0699 90)
@@
 		)
 		(property "Value" "PESD0402-140"
-			(at 59.69 181.6099 90)
+			(at 60.198 172.466 90)
 			(effects
 				(font
@@
 			)
 		)
-		(property "Value" "D_Schottky"
+		(property "Value" "MBRA160T3G"
 			(at 187.0075 21.59 0)
 			(effects
