File: FLP_PCB/FLP_PCB_terminal/mistance_PCB_terminal.kicad_sch (KiCad schematic)
At the start: 65 parts, among them J1 SMA-J-P-X-ST-TH1, Q1 Q_PMOS_DSG, Q2 UMH3N, U1 AMS1117-3.3, U2 L86-M33, U3 STM32F103C8T6, U4 MCP73831-2-OT, U5 CP2104, U6 TPS61200DRC, U7 USBLC6-2P6, U8 SX1278, Y1 Crystal, Y2 ABM3B-8.000MHZ-B2-T

Commit message: dir name change, host PCB finish
Parts:
- removed Q2: UMH3N, Package_TO_SOT_SMD:SOT-363_SC-70-6, symbol Transistor_BJT:UMH3N
- removed R5, R6: 10K, Resistor_SMD:R_0603_1608Metric, symbol Device:R
- added C26: 4.7uF, Capacitor_SMD:C_0603_1608Metric, symbol Device:C
- added C27: 0.1uF, Capacitor_SMD:C_0603_1608Metric, symbol Device:C
- added C28, C29: PESD0402-140, PESD0402-140:RESC1005X35N, symbol PESD0402-140:PESD0402-140
- added Find_Host, ID: SKRPABE010, Diode_SMD:SW_SKRPABE010, symbol SKRPABE010:SKRPABE010
- added J4: OLED, HTSW-104-20-TM-S:SAMTEC_HTSW-104-20-TM-S, symbol HTSW-104-20-TM-S:HTSW-104-20-TM-S
- added R17, R18, R21: 10K, Resistor_SMD:R_0603_1608Metric, symbol Device:R
- added R19, R20: 2.2K, Resistor_SMD:R_0603_1608Metric, symbol Device:R
- added R7: 1K, Resistor_SMD:R_0603_1608Metric, symbol Device:R
- BZ1: footprint (none) -> Buzzer_Beeper:Buzzer_15x7.5RM7.6
- renumbered C7 to C10, C8 to C11, C9 to C12, C10 to C13, C11 to C14, C12 to C15, C13 to C16, C14 to C17, C15 to C18, C16 to C19, C17 to C20, C18 to C21, C19 to C22, C20 to C23, C22 to C24, C24 to C25, C5 to C3, C3 to C4, C4 to C5, C23 to C6, C25 to C7, C6 to C8, C21 to C9, Q1 to Q2, R16 to R1, R8 to R10, R15 to R11, R9 to R12, R10 to R13, R11 to R14, R12 to R15, R13 to R16, R14 to R2, R1 to R3, R2 to R4, R3 to R5, R4 to R6, R7 to R9, S2 to S1, S1 to S2, U3 to U2, U2 to U3, Y2 to Y1, Y1 to Y2
Connections:
- net 3.3V OUT: now also C26.1, C27.1, Find_Host.1, Find_Host.2, ID.1, ID.2, J4.02, R19.2, R20.2
- net BOOT0: now also S1.1, S1.2
- net GND: now also C26.2, C27.2, C28.2, C29.2, J4.01, R17.1, R18.1, R21.1; no longer S1.1, S1.2
- net at C3.1, Charger1.1 (VBUS), D1.2 (A)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: now also R7.1; no longer Q2.3 (G)
- net at U2.20 (PB2): now also R21.2
- net Find_Host: now reaches U2.39 (PB3)
- net Find_Host: now also Find_Host.3, Find_Host.4, R18.2
- net ID: now reaches U2.40 (PB4)
- net ID: now also ID.3, ID.4, R17.2
- net I2C SCL: now reaches U2.42 (PB6)
- net I2C SCL: now also C29.1, J4.03, R20.1
- net I2C SDL: now reaches U2.43 (PB7)
- net I2C SDL: now also C28.1, J4.04, R19.1
- new net: Q2.3 (G), R7.2
- no-connect marks 50 -> 47
