File: FLP_PCB/FLP_PCB_terminal/FLP_PCB_terminal.kicad_sch (KiCad schematic)
At the start: 75 parts, among them J1 SMA-J-P-X-ST-TH1, J4 OLED, Q2 Q_PMOS_DSG, U1 AMS1117-3.3, U2 STM32F103C8T6, U3 L86-M33, U4 MCP73831-2-OT, U5 CP2104, U6 TPS61200DRC, U7 USBLC6-2P6, U8 SX1278, Y1 ABM3B-8.000MHZ-B2-T, Y2 Crystal

Commit message: modify
Parts:
- added C30, C31, C32: 0.1uF, Capacitor_SMD:C_0603_1608Metric, symbol Device:C
- added Y3: 32.768kHz, Crystal:Crystal_SMD_3215-2Pin_3.2x1.5mm, symbol Device:Crystal
- Y2: value Crystal -> 32MHz
- renumbered C28 to C21, C29 to C22, C26 to C23, C27 to C24, C21 to C25, C22 to C26, C23 to C27, C24 to C28, C25 to C29, Find_Host to Find_Host1, ID to ID1, J4 to J2, Q2 to Q1, R7 to R10, R19 to R15, R15 to R16, R16 to R17, R20 to R18, R17 to R19, R18 to R20, R21 to R5, R5 to R6, R6 to R7, R9 to R8, R10 to R9
Connections:
- net 3.3V OUT: no longer U2.1 (VBAT)
- net 5v OUT: now also FL1.2, UART1.A4 (VBUS), UART1.A9 (VBUS), UART1.B4 (VBUS), UART1.B9 (VBUS)
- net GND: now also C30.2, C31.2, C32.1
- net NRST: now also C32.2
- net RX: now also U2.31 (PA10); no longer U2.30 (PA9)
- net TX: now also U2.30 (PA9); no longer U2.31 (PA10)
- net PC_OSC_IN: now reaches U2.3 (PC14-OSC32_IN)
- net PC_OSC_IN: now also C31.1, Y3.1
- net PC_OSC_OUT: now reaches U2.4 (PC15-OSC32_OUT)
- net PC_OSC_OUT: now also C30.1, Y3.2
- net PB0: no longer names the net of U2.18 (PB0)
Other:
- moved on the sheet: BZ1, C9

Commit message: PCB
Parts:
- Y2: footprint Crystal:Crystal_SMD_2012-2Pin_2.0x1.2mm -> Crystal:Crystal_SMD_2016-4Pin_2.0x1.6mm
Changed lines of the file:
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@@
 			)
 		)
-		(property "Footprint" "Crystal:Crystal_SMD_2012-2Pin_2.0x1.2mm"
+		(property "Footprint" "Crystal:Crystal_SMD_2016-4Pin_2.0x1.6mm"
 			(at 231.14 77.47 0)
 			(effects

Commit message: code adding
Parts:
- BZ1: footprint Buzzer_Beeper:Buzzer_15x7.5RM7.6 -> Buzzer_Beeper:Buzzer_12x9.5RM7.6
Changed lines of the file:
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@@
 			)
 		)
-		(property "Footprint" "Buzzer_Beeper:Buzzer_15x7.5RM7.6"
+		(property "Footprint" "Buzzer_Beeper:Buzzer_12x9.5RM7.6"
 			(at 120.015 78.74 90)
 			(effects
