File: FLP_device_PCB/FLP_PCB_terminal/FLP_PCB_terminal.kicad_pcb (KiCad board)
At the start: 4 copper layers, 80 x 80 mm, 79 parts, among them J1 SMA-J-P-X-ST-TH1, J2 OLED, Q1 Q_PMOS_DSG, U1 AMS1117-3.3, U2 STM32F103C8T6, U3 L86-M33, U4 MCP73831-2-OT, U5 CP2104, U6 TPS61200DRC, U7 USBLC6-2P6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

Commit message: device_code fix and device_PCB fix
Parts:
- C27: value 27pF -> 2.2pF
Connections:
- D1 pad A: 5v OUT -> (no net)
- D1 pad C: Net-(Charger1-VBUS) -> (no net)
- UART1 pad A1_B12: GND -> (no net)
- UART1 pad B1_A12: GND -> (no net)
- Y2 pad 1: (no net) -> Net-(U8-XTB)
- Y2 pad 4: Net-(U8-XTB) -> (no net)
Changed lines of the file:
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@@
 			(size 2.3 1.55)
 			(layers "F.Cu" "F.Mask" "F.Paste")
-			(net 4 "5v OUT")
 			(solder_mask_margin 0.102)
 		)
@@
 			(size 2.3 1.55)
 			(layers "F.Cu" "F.Mask" "F.Paste")
-			(net 6 "Net-(Charger1-VBUS)")
 			(solder_mask_margin 0.102)
 		)
@@
 			(size 0.9 0.8)
 			(layers "F.Cu" "F.Mask" "F.Paste")
+			(net 15 "Net-(U8-XTB)")
 			(pinfunction "1")
 			(pintype "passive")
@@
 			(size 0.9 0.8)
 			(layers "F.Cu" "F.Paste")
-			(net 15 "Net-(U8-XTB)")
 		)
 		(embedded_fonts no)
@@
 			)
 		)
-		(property "Value" "27pF"
+		(property "Value" "2.2pF"
 			(at 0 1.43 0)
 			(layer "F.Fab")
@@
 			(size 0.6 0.98)
 			(layers "F.Cu" "F.Mask" "F.Paste")
-			(net 2 "GND")
 			(solder_mask_margin 0.09)
 		)
@@
 			(size 0.6 0.98)
 			(layers "F.Cu" "F.Mask" "F.Paste")
-			(net 2 "GND")
 			(solder_mask_margin 0.09)
 		)
@@
 			)
 		)
-		(property "Description" ""
+		(property "Description" "Buzzer, polarized"
 			(at 0 0 0)
 			(unlocked yes)
