File: FLP_device_PCB/FLP_PCB_terminal/FLP_PCB_terminal.kicad_sch (KiCad schematic)
At the start: 79 parts, among them J1 SMA-J-P-X-ST-TH1, J2 OLED, Q1 Q_PMOS_DSG, U1 AMS1117-3.3, U2 STM32F103C8T6, U3 L86-M33, U4 MCP73831-2-OT, U5 CP2104, U6 TPS61200DRC, U7 USBLC6-2P6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

Commit message: device_code fix and device_PCB fix
Parts:
- C27: value 27pF -> 2.2pF
Changed lines of the file:
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@@
 			)
 		)
-		(property "Description" ""
+		(property "Description" "744028000056"
 			(at 252.73 16.51 0)
 			(effects
@@
 			)
 		)
-		(property "Value" "27pF"
+		(property "Value" "2.2pF"
 			(at 237.49 11.43 90)
 			(effects

Commit message: FLP_set add
Other:
- moved on the sheet: R5
Changed lines of the file:
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@@
 	(wire
 		(pts
-			(xy 88.9 106.68) (xy 87.63 107.95)
+			(xy 90.17 106.68) (xy 87.63 107.95)
 		)
 		(stroke
@@
 	(wire
 		(pts
+			(xy 90.17 97.79) (xy 88.9 97.79)
+		)
+		(stroke
+			(width 0)
+			(type default)
+		)
+	)
+	(wire
+		(pts
 			(xy 121.92 73.66) (xy 140.97 73.66)
 		)
@@
 	(wire
 		(pts
+			(xy 88.9 97.79) (xy 88.9 95.25)
+		)
+		(stroke
+			(width 0)
+			(type default)
+		)
+	)
+	(wire
+		(pts
 			(xy 19.05 91.44) (xy 25.4 97.79)
 		)
@@
 	(wire
 		(pts
-			(xy 88.9 95.25) (xy 88.9 99.06)
+			(xy 90.17 97.79) (xy 90.17 99.06)
 		)
 		(stroke
@@
 	(symbol
 		(lib_id "Device:R")
-		(at 88.9 102.87 0)
+		(at 90.17 102.87 0)
 		(unit 1)
 		(exclude_from_sim no)
@@
 		(fields_autoplaced yes)
 		(property "Reference" "R5"
-			(at 91.44 101.5999 0)
+			(at 92.71 101.5999 0)
 			(effects
 				(font
@@
 		)
 		(property "Value" "10K"
-			(at 91.44 104.1399 0)
+			(at 92.71 104.1399 0)
 			(effects
 				(font
@@
 		)
 		(property "Footprint" "Resistor_SMD:R_0603_1608Metric"
-			(at 87.122 102.87 90)
+			(at 88.392 102.87 90)
 			(effects
 				(font
@@
 		)
 		(property "Datasheet" "~"
-			(at 88.9 102.87 0)
+			(at 90.17 102.87 0)
 			(effects
 				(font
@@
 		)
 		(property "Description" "Resistor"
-			(at 88.9 102.87 0)
+			(at 90.17 102.87 0)
 			(effects
 				(font
