File: FLP_device_PCB/FLP_PCB_set/FLP_PCB_set/LoRa.kicad_sch (KiCad schematic)
At the start: 11 parts, among them J8 SMA-J-P-X-ST-TH1, U13 SX1278, Y2 32MHz

Commit message: PCB fixing end adding description pdf
Parts:
- L3, L4: footprint Capacitor_SMD:C_0402_1005Metric -> Inductor_SMD:L_0402_1005Metric
Changed lines of the file:
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@@
 			)
 		)
-		(property "Footprint" "Capacitor_SMD:C_0402_1005Metric"
+		(property "Footprint" "Inductor_SMD:L_0402_1005Metric"
 			(at 73.66 30.48 0)
 			(effects
@@
 			)
 		)
-		(property "Footprint" "Capacitor_SMD:C_0402_1005Metric"
+		(property "Footprint" "Inductor_SMD:L_0402_1005Metric"
 			(at 81.28 26.67 0)
 			(effects
