File: FLP_device_PCB/FLP_PCB_set/FLP_PCB_set/STM32.kicad_sch (KiCad schematic)
At the start: 1 part, among them U9 STM32F103C8T6

Commit message: FLP_set add
Parts:
- added BZ1: Buzzer, Buzzer_Beeper:Buzzer_12x9.5RM7.6, symbol Device:Buzzer
- added C36: 0.1uF, Capacitor_SMD:C_0603_1608Metric, symbol Device:C
- added C37: 1uF, Capacitor_SMD:C_0603_1608Metric, symbol Device:C
- added C38, C39: 20pF, Capacitor_SMD:C_0402_1005Metric, symbol Device:C
- added C40, C41: 18pF, Capacitor_SMD:C_0603_1608Metric, symbol Device:C
- added Find_Host2, ID1, S2: SKRPABE010, Diode_SMD:SW_SKRPABE010, symbol SKRPABE010:SKRPABE010
- added R26, R28, R29: 10K, Resistor_SMD:R_0603_1608Metric, symbol Device:R
- added R27: 1M, Resistor_SMD:R_0603_1608Metric, symbol Device:R
- added Y3: ABM3B-8.000MHZ-B2-T, ABM3B-8.000MHZ-B2-T:XTAL_ABM3B-8.000MHZ-B2-T, symbol ABM3B-8.000MHZ-B2-T:ABM3B-8.000MHZ-B2-T
- added Y4: 32.768kHz, Crystal:Crystal_SMD_3215-2Pin_3.2x1.5mm, symbol Device:Crystal
Connections:
- net 3.3V_in: now also R26.1
- net VBAT: now reaches U9.1 (VBAT)
- net GPS_Reset: now reaches U9.11 (PA1)
- net GPS_Rx: now reaches U9.12 (PA2)
- net GPS_TX: now reaches U9.13 (PA3)
- net NSS(CS): now reaches U9.14 (PA4)
- net SCK: now reaches U9.15 (PA5)
- net MISO: now reaches U9.16 (PA6)
- net MOSI: now reaches U9.17 (PA7)
- net DIO0(IRQ): now reaches U9.19 (PB1)
- net BOOT1: now reaches U9.20 (PB2)
- net GND: now reaches U9.23 (VSS), U9.35 (VSS), U9.47 (VSS)
- net GND: now also U9.8 (VSSA), BZ1.2 (-), C36.1, C37.2, C40.2, C41.2, R28.2, R29.2, S2.3, S2.4, Y3.2 (GND), Y3.4 (GND)
- net RESET: now reaches U9.29 (PA8)
- net PC_OSC_IN: now reaches U9.3 (PC14-OSC32_IN)
- net PC_OSC_IN: now also C41.1, Y4.1
- net Buzzer: now reaches U9.32 (PA11)
- net Buzzer: now also BZ1.1 (+), C37.1
- net ID: now reaches U9.39 (PB3)
- net ID: now also ID1.3, ID1.4, R28.1
- net PC_OSC_OUT: now reaches U9.4 (PC15-OSC32_OUT)
- net PC_OSC_OUT: now also C40.1, Y4.2
- net Find_Host: now reaches U9.40 (PB4)
- net Find_Host: now also Find_Host2.3, Find_Host2.4, R29.1
- net BOOT0: now reaches U9.44 (BOOT0)
- net OSC_IN: now reaches U9.5 (PD0_OSC_IN)
- net OSC_IN: now also C38.2, R27.1, Y3.3
- net OSC_OUT: now reaches U9.6 (PD1_OSC_OUT)
- net OSC_OUT: now also C39.2, R27.2, Y3.1
- net at U9.7 (NRST): now also C36.2, R26.2, S2.1, S2.2
- new net: C38.1, C39.1
- new net 3.3V_OUT: Find_Host2.1, Find_Host2.2, ID1.1, ID1.2
- no-connect marks 0 -> 18

Commit message: PCB fixing end adding description pdf
Parts:
- BZ1: value Buzzer -> FQ 010
Connections:
- net 3.3V_OUT is gone; now on net 3.3V_in: Find_Host2.1, Find_Host2.2, ID1.1, ID1.2
Changed lines of the file:
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@@
-		)
-	)
-	(hierarchical_label "3.3V_OUT"
-		(shape output)
-		(at 157.48 127 180)
-		(effects
-			(font
-				(size 1.27 1.27)
-			)
-			(justify right)
 		)
 	)
@@
 		)
 	)
+	(hierarchical_label "3.3V_in"
+		(shape output)
+		(at 157.48 116.84 180)
+		(effects
+			(font
+				(size 1.27 1.27)
+			)
+			(justify right)
+		)
+	)
 	(hierarchical_label "TX"
 		(shape input)
@@
 		)
 	)
-	(hierarchical_label "3.3V_OUT"
+	(hierarchical_label "3.3V_in"
 		(shape output)
-		(at 157.48 116.84 180)
+		(at 157.48 127 180)
 		(effects
 			(font
@@
 		)
 		(instances
-			(project ""
+			(project "FLP_PCB_set"
 				(path "/3f8c5218-62bd-4afc-a38b-629e4a961e52/cb21122d-83f9-4f10-9012-eb16f816aa97/0ae67f6e-4f17-4cbc-bbf5-63c02f98d1d0"
 					(reference "#PWR040")
@@
 			)
 		)
-		(property "Value" "Buzzer"
+		(property "Value" "FQ 010"
 			(at 157.226 63.246 0)
 			(effects
