File: FLP_device_PCB/FLP_PCB_set/FLP_PCB_set/USB_CC.kicad_sch (KiCad schematic)
At the start: 2 parts

Commit message: FLP_set add
Parts:
- removed R18: 5K, symbol Device:R
- added R21: 5.1K, symbol Device:R
- R20: renamed from R17; value 5K -> 5.1K
Connections:
- net CC_2: now also R21.1
- net GND: now also R21.2
Changed lines of the file:
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@@
 		(dnp no)
 		(fields_autoplaced yes)
-		(property "Reference" "R17"
+		(property "Reference" "R20"
 			(at 24.13 29.2099 0)
 			(effects
@@
 			)
 		)
-		(property "Value" "5K"
+		(property "Value" "5.1K"
 			(at 24.13 31.7499 0)
 			(effects
@@
 			(project ""
 				(path "/3f8c5218-62bd-4afc-a38b-629e4a961e52/cb21122d-83f9-4f10-9012-eb16f816aa97/2508fd1a-b460-4e54-ae43-854b285e1d14"
-					(reference "R17")
+					(reference "R20")
 					(unit 1)
 				)
@@
 		(dnp no)
 		(fields_autoplaced yes)
-		(property "Reference" "#PWR032"
+		(property "Reference" "#PWR031"
 			(at 21.59 44.45 0)
 			(effects
@@
 			(project ""
 				(path "/3f8c5218-62bd-4afc-a38b-629e4a961e52/cb21122d-83f9-4f10-9012-eb16f816aa97/2508fd1a-b460-4e54-ae43-854b285e1d14"
-					(reference "#PWR032")
+					(reference "#PWR031")
 					(unit 1)
 				)
@@
 		(dnp no)
 		(fields_autoplaced yes)
-		(property "Reference" "R18"
+		(property "Reference" "R21"
 			(at 33.02 29.2099 0)
 			(effects
@@
 			)
 		)
-		(property "Value" "5K"
+		(property "Value" "5.1K"
 			(at 33.02 31.7499 0)
 			(effects
@@
 			(project "FLP_PCB_set"
 				(path "/3f8c5218-62bd-4afc-a38b-629e4a961e52/cb21122d-83f9-4f10-9012-eb16f816aa97/2508fd1a-b460-4e54-ae43-854b285e1d14"
-					(reference "R18")
+					(reference "R21")
 					(unit 1)
 				)

Commit message: PCB fixing end adding description pdf
Parts:
- R20, R21: footprint (none) -> Resistor_SMD:R_0603_1608Metric
Changed lines of the file:
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@@
 			)
 		)
-		(property "Footprint" ""
+		(property "Footprint" "Resistor_SMD:R_0603_1608Metric"
 			(at 19.812 30.48 90)
 			(effects
@@
 		)
 		(instances
-			(project ""
+			(project "FLP_PCB_set"
 				(path "/3f8c5218-62bd-4afc-a38b-629e4a961e52/cb21122d-83f9-4f10-9012-eb16f816aa97/2508fd1a-b460-4e54-ae43-854b285e1d14"
 					(reference "R20")
@@
 		)
 		(instances
-			(project ""
+			(project "FLP_PCB_set"
 				(path "/3f8c5218-62bd-4afc-a38b-629e4a961e52/cb21122d-83f9-4f10-9012-eb16f816aa97/2508fd1a-b460-4e54-ae43-854b285e1d14"
 					(reference "#PWR031")
@@
 			)
 		)
-		(property "Footprint" ""
+		(property "Footprint" "Resistor_SMD:R_0603_1608Metric"
 			(at 28.702 30.48 90)
 			(effects
