File: FLP_device_PCB/FLP_PCB_set/FLP_PCB_set/FLP_host.kicad_sch (KiCad schematic)
At the start: 82 parts, among them J3 GRPB052VWVN-RC, J4 OLED, J5 SMA-J-P-X-ST-TH1, Q1 Q_PMOS_DSG, Q2 UMH3N, U1 ESP32-WROOM-32E, U2 TPS61200DRC, U3 MCP73831-2-OT, U4 AMS1117-3.3, U5 CP2104, U6 L86-M33, U7 SX1278, U8 USBLC6-2P6, Y1 32MHz

Commit message: FLP_set add
Parts:
- removed BT1: Battery_Cell, Battery:BatteryHolder_MPD_BH-18650-PC2, symbol Device:Battery_Cell
- removed C10, C32, C4, C5, C9: 4.7uF, Capacitor_SMD:C_0603_1608Metric, symbol Device:C
- removed C11, C29, C31, C33: 22uF, Capacitor_SMD:C_0805_2012Metric, symbol Device:C
- removed C28, C30: 0.1uF, Capacitor_SMD:C_0603_1608Metric, symbol Device:C
- removed C34: 1uF, Capacitor_SMD:C_0603_1608Metric, symbol Device:C
- removed D1: MBRA160T3G, Diode_SMD:DIOM5226X220N, symbol Device:D_Schottky
- removed F1: 0603L100SLYR, Resistor_SMD:R_0603_1608Metric, symbol Device:Polyfuse
- removed FL1: BLM21PG221SN1D, BLM21PG221SN1D:BEADC2012X105N, symbol BLM21PG221SN1D:BLM21PG221SN1D
- removed L4: 744028000056, WE-TPC_2811:WE-TPC_2811, symbol WE-TPC_2811:WE-TPC_2811
- removed Q1: Q_PMOS_DSG, SI2333DS-T1-E3:SOT95P237X112-3N, symbol Transistor_FET:Q_PMOS_DSG
- removed R1: 2M, Resistor_SMD:R_1210_3225Metric, symbol Device:R
- removed R2: 180K, Resistor_SMD:R_1210_3225Metric, symbol Device:R
- removed R22, R3, R4: 10K, Resistor_SMD:R_0603_1608Metric, symbol Device:R
- removed R23, R31: 1K, Resistor_SMD:R_0603_1608Metric, symbol Device:R
- removed R25, R29: 100R, Resistor_SMD:R_0603_1608Metric, symbol Device:R
- removed R5: 100R, Resistor_SMD:R_0402_1005Metric, symbol Device:R
- removed R6: 22R, Resistor_SMD:R_0402_1005Metric, symbol Device:R
- removed U2: TPS61200DRC, Package_SON:Texas_S-PVSON-N10_ThermalVias, symbol Regulator_Switching:TPS61200DRC
- removed U3: MCP73831-2-OT, Package_TO_SOT_SMD:SOT95P280X145-5N, symbol Battery_Management:MCP73831-2-OT
- removed U4: AMS1117-3.3, Package_TO_SOT_SMD:SOT-223-3_TabPin2, symbol Regulator_Linear:AMS1117-3.3
- removed U5: CP2104, Package_DFN_QFN:QFN-24-1EP_4x4mm_P0.5mm_EP2.6x2.6mm, symbol Interface_USB:CP2104
- removed UART1: 12402012E212A, 12402012E212A:AMPHENOL_12402012E212A, symbol Connector:USB_C_Receptacle_USB2.0_16P
- added C14, C18: 22uF, Capacitor_SMD:C_0805_2012Metric, symbol Device:C
- added C17: 10uF, Capacitor_SMD:C_0805_2012Metric, symbol Device:C
- added C24: 3.3pF, Capacitor_SMD:C_0402_1005Metric, symbol Device:C
- added D1: MBR120VLSFT1G, MBR120VLSFT1G:DIOM3616X98N, symbol MBR120VLSFT1G:MBR120VLSFT1G
- added D2: BAT ON, LED_SMD:LED_0805_2012Metric, symbol Device:LED
- added D3: TEST, LED_SMD:LED_0805_2012Metric, symbol Device:LED
- added D4: USB_ON, LED_SMD:LED_0805_2012Metric, symbol Device:LED
- added J3: B2B-PH-K-S, B2B_PH_K_S:JST_B2B-PH-K-S, symbol B2B-PH-K-S:B2B-PH-K-S
- added J4: USB_C_Receptacle_USB2.0_16P, 12402012E212A:AMPHENOL_12402012E212A, symbol Connector:USB_C_Receptacle_USB2.0_16P
- added L2: 18nH, Capacitor_SMD:C_0402_1005Metric, symbol Device:L
- added Q1: DMG3415UQ-7, symbol DMG3415UQ-7:DMG3415UQ-7
- added R12: 100K, Resistor_SMD:R_0603_1608Metric, symbol Device:R
- added R13: 2K, Resistor_SMD:R_0402_1005Metric, symbol Device:R
- added R14, R15: 1K, Resistor_SMD:R_0603_1608Metric, symbol Device:R
- added U3: AP2112K-3.3, Package_TO_SOT_SMD:SOT-23-5, symbol Regulator_Linear:AP2112K-3.3
- added U4: CP2104, Package_DFN_QFN:QFN-24-1EP_4x4mm_P0.5mm_EP2.6x2.6mm, symbol Interface_USB:CP2104
- added U5: MCP73831-2-OT, Package_TO_SOT_SMD:SOT-23-5, symbol Battery_Management:MCP73831-2-OT
- C21: renamed from C20; value 27pF -> 15pF; footprint Capacitor_SMD:C_0603_1608Metric -> Capacitor_SMD:C_0402_1005Metric
- L1: value 2.2uH -> 47nH; footprint Inductor_SMD:L_1210_3225Metric -> Capacitor_SMD:C_0402_1005Metric
- R7: value 22R -> 100K; footprint Resistor_SMD:R_0402_1005Metric -> Resistor_SMD:R_0603_1608Metric
- renumbered C37 to C1, C6 to C10, C16 to C11, C18 to C12, C19 to C13, C17 to C15, C12 to C16, C22 to C19, C27 to C2, C21 to C20, C23 to C22, C24 to C23, C8 to C3, C13 to C4, C14 to C5, C15 to C6, C35 to C8, C25 to C9, J3 to J1, J4 to J2, R10 to R1, R33 to R10, R15 to R11, R8 to R16, R21 to R17, R20 to R18, R16 to R19, R11 to R2, R12 to R3, R13 to R4, R30 to R5, R9 to R6, R14 to R8, R32 to R9, U6 to U1, U1 to U2, U8 to U6
Connections:
- net 3.3V_OUT: now also J2.03, U6.2 (GND), C17.1, U3.5 (VOUT), U4.5 (VIO), U4.6 (VDD), U4.7 (REGIN); no longer J2.02
- net Ctrl: now also Ctrl1.3, Ctrl1.4, R18.1
- net DTR: now also U4.23 (~{DTR})
- net Find_Host: now also Find_Host1.3, Find_Host1.4, R19.1
- net GND: now also C4.1, C5.1, J2.04, L1.1, R7.2, U6.5 (VBUS), C14.2, C17.2, C18.2, C24.2, J3.2, J4.A12 (GND), J4.A1_B12 (GND), J4.B1 (GND), J4.B12 (GND), J4.B1_A12 (GND), J4.SH1 (SHIELD), J4.SH2 (SHIELD), J4.SH3 (SHIELD), J4.SH4 (SHIELD), R13.1, R14.2, U3.2 (GND), U4.2 (GND), U4.25 (GND), U5.2 (V_{SS}); no longer C4.2, C5.2, J2.01, U6.2 (GND)
- net GPS_Reset: now also U1.10 (~{RESET})
- net I2C_SCL: now also J2.01; no longer J2.03
- net I2C_SDL: now also J2.02; no longer J2.04
- net RTS: now also U4.19 (~{RTS})
- net RX: now also U4.21 (TXD); no longer R7.1
- net TX: now also U4.20 (RXD)
- net at R16.2: now also J4.B5 (CC2)
- net at C21.2: now also J5.1
- net at U7.27 (PA_BOOST): now also C24.1, L2.2
- net at U6.1 (I/O1): now also J4.A7 (D-), J4.B7 (D-)
- net at U6.3 (I/O2): now also J4.A6 (D+), J4.B6 (D+)
- net at U6.4 (I/O2): now also U4.3 (D+)
- net at U6.6 (I/O1): now also U4.4 (D-)
- net at J1.6, R2.2: now also C5.2; no longer C5.1
- net at L1.2: now also C21.1, L2.1
- net at R17.2: now also J4.A5 (CC1)
- net at J1.4, R3.2: now also C4.2; no longer C4.1
- net TEST LED: now reaches U2.7 (IO35)
- net TEST LED: now also D3.2 (A)
- new net: C14.1, D1.1, D2.1 (K), D2.2 (A), Q1.2 (S), R12.2, U3.1 (VIN)
- new net: D3.1 (K), R14.1
- new net: R12.1, U3.3 (EN)
- new net: R13.2, U5.5 (PROG)
- new net: D4.1 (K), R15.2
- new net: R15.1, U5.1 (STAT)
- new net 5v_USB_OUT: D1.2, D4.2 (A), J4.A4_B9 (VBUS), J4.A9 (VBUS), J4.B4 (VBUS), J4.B4_A9 (VBUS), J4.B9 (VBUS), Q1.1 (G), R7.1, U4.8 (VBUS), U5.4 (V_{DD})
- new net VBAT: C18.1, J3.1, Q1.3 (D), U5.3 (V_{BAT})
Other:
- moved on the sheet: C12, C13, C16, C21, C3, C4, C5, C6, C7, C9, Ctrl1, Find_Host1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

Commit message: PCB fixing end adding description pdf
Parts:
- removed D2: BAT ON, LED_SMD:LED_0805_2012Metric, symbol Device:LED
- D3: value TEST -> 150080GS75000
- D4: value USB_ON -> 150080GS75000
- J4: value USB_C_Receptacle_USB2.0_16P -> 12402012E212A
- L1: footprint Capacitor_SMD:C_0402_1005Metric -> Inductor_SMD:L_0402_1005Metric
Connections:
- net 3.3V_OUT: no longer U6.2 (GND)
- net 5v_USB_OUT: now also U6.5 (VBUS)
- net GND: now also U6.2 (GND); no longer U6.5 (VBUS)
Changed lines of the file:
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@@
 	)
 	(junction
-		(at 114.3 35.56)
-		(diameter 0)
-		(color 0 0 0 0)
-	)
-	(junction
 		(at 264.16 137.16)
 		(diameter 0)
@@
 	)
 	(junction
-		(at 187.96 130.81)
-		(diameter 0)
-		(color 0 0 0 0)
-	)
-	(junction
 		(at 196.85 132.08)
 		(diameter 0)
@@
 	)
 	(junction
-		(at 124.46 39.37)
-		(diameter 0)
-		(color 0 0 0 0)
-	)
-	(junction
 		(at 97.79 46.99)
 		(diameter 0)
@@
 	(wire
 		(pts
-			(xy 185.42 130.81) (xy 187.96 130.81)
-		)
-		(stroke
-			(width 0)
-			(type default)
-		)
-	)
-	(wire
-		(pts
 			(xy 210.82 88.9) (xy 213.36 88.9)
 		)
@@
 	(wire
 		(pts
-			(xy 185.42 121.92) (xy 185.42 130.81)
+			(xy 185.42 121.92) (xy 185.42 128.27)
 		)
 		(stroke
@@
 	(wire
 		(pts
+			(xy 185.42 95.25) (xy 189.23 95.25)
+		)
+		(stroke
+			(width 0)
+			(type default)
+		)
+	)
+	(wire
+		(pts
 			(xy 251.46 67.31) (xy 251.46 74.93)
 		)
@@
 	(wire
 		(pts
+			(xy 189.23 95.25) (xy 189.23 97.79)
+		)
+		(stroke
+			(width 0)
+			(type default)
+		)
+	)
+	(wire
+		(pts
 			(xy 264.16 160.02) (xy 264.16 162.56)
 		)
@@
 	(wire
 		(pts
-			(xy 124.46 35.56) (xy 123.19 35.56)
-		)
-		(stroke
-			(width 0)
-			(type default)
-		)
-	)
-	(wire
-		(pts
 			(xy 242.57 110.49) (xy 251.46 110.49)
 		)
@@
 	(wire
 		(pts
-			(xy 115.57 35.56) (xy 114.3 35.56)
-		)
-		(stroke
-			(width 0)
-			(type default)
-		)
-	)
-	(wire
-		(pts
 			(xy 236.22 67.31) (xy 238.76 67.31)
 		)
@@
 	(wire
 		(pts
-			(xy 124.46 35.56) (xy 124.46 39.37)
-		)
-		(stroke
-			(width 0)
-			(type default)
-		)
-	)
-	(wire
-		(pts
 			(xy 71.12 99.06) (xy 67.31 99.06)
 		)
@@
 	(hierarchical_label "5v_USB_OUT"
 		(shape output)
+		(at 185.42 128.27 270)
+		(effects
+			(font
+				(size 1.27 1.27)
+			)
+			(justify right)
+		)
+	)
+	(hierarchical_label "5v_USB_OUT"
+		(shape output)
 		(at 97.79 25.4 90)
 		(effects
@@
 		)
 	)
-	(hierarchical_label "3.3V_OUT"
-		(shape output)
-		(at 185.42 95.25 90)
-		(effects
-			(font
-				(size 1.27 1.27)
-			)
-			(justify left)
-		)
-	)
 	(hierarchical_label "DTR"
 		(shape bidirectional)
@@
 	)
 	(symbol
-		(lib_id "Device:LED")
-		(at 119.38 35.56 180)
-		(unit 1)
-		(exclude_from_sim no)
-		(in_bom yes)
-		(on_board yes)
-		(dnp no)
-		(property "Reference" "D2"
-			(at 119.888 30.48 0)
-			(effects
-				(font
-					(size 1.27 1.27)
-				)
-			)
-		)
-		(property "Value" "BAT ON"
-			(at 119.888 33.02 0)
-			(effects
-				(font
-					(size 1.27 1.27)
-				)
-			)
-		)
-		(property "Footprint" "LED_SMD:LED_0805_2012Metric"
-			(at 119.38 35.56 0)
-			(effects
-				(font
-					(size 1.27 1.27)
-				)
-				(hide yes)
-			)
-		)
-		(property "Datasheet" "~"
-			(at 119.38 35.56 0)
-			(effects
-				(font
-					(size 1.27 1.27)
-				)
-				(hide yes)
-			)
-		)
-		(property "Description" "Light emitting diode"
-			(at 119.38 35.56 0)
-			(effects
-				(font
-					(size 1.27 1.27)
-				)
-				(hide yes)
-			)
-		)
-		(property "Sim.Pins" "1=K 2=A"
-			(at 119.38 35.56 0)
-			(effects
-				(font
-					(size 1.27 1.27)
-				)
-				(hide yes)
-			)
-		)
-		(pin "1"
-		)
-		(pin "2"
-		)
-		(instances
-			(project "FLP_PCB_set"
-				(path "/3f8c5218-62bd-4afc-a38b-629e4a961e52/3028588a-b9cc-4609-a7ce-985f9df6b777"
-					(reference "D2")
-					(unit 1)
-				)
-			)
-		)
-	)
-	(symbol
 		(lib_id "SKRPABE010:SKRPABE010")
 		(at 245.11 149.86 0)
@@
 		(on_board yes)
 		(dnp no)
+		(fields_autoplaced yes)
 		(property "Reference" "Q1"
 			(at 117.856 24.384 0)
@@
 		(on_board yes)
 		(dnp no)
+		(fields_autoplaced yes)
 		(property "Reference" "R12"
 			(at 121.412 37.592 90)
@@
 			)
 		)
-		(property "Value" "TEST"
+		(property "Value" "150080GS75000"
 			(at 156.718 185.42 0)
 			(effects
@@
 		(on_board yes)
 		(dnp no)
+		(fields_autoplaced yes)
 		(property "Reference" "R7"
 			(at 102.87 44.704 0)
@@
 	)
 	(symbol
+		(lib_id "power:GND")
+		(at 189.23 97.79 0)
+		(unit 1)
+		(exclude_from_sim no)
+		(in_bom yes)
+		(on_board yes)
+		(dnp no)
+		(fields_autoplaced yes)
+		(property "Reference" "#PWR058"
+			(at 189.23 104.14 0)
+			(effects
+				(font
+					(size 1.27 1.27)
+				)
+				(hide yes)
+			)
+		)
+		(property "Value" "GND"
+			(at 189.23 102.87 0)
+			(effects
+				(font
+					(size 1.27 1.27)
+				)
+			)
+		)
+		(property "Footprint" ""
+			(at 189.23 97.79 0)
+			(effects
+				(font
+					(size 1.27 1.27)
+				)
+				(hide yes)
+			)
+		)
+		(property "Datasheet" ""
+			(at 189.23 97.79 0)
+			(effects
+				(font
+					(size 1.27 1.27)
+				)
+				(hide yes)
+			)
+		)
+		(property "Description" "Power symbol creates a global label with name \"GND\" , ground"
+			(at 189.23 97.79 0)
+			(effects
+				(font
+					(size 1.27 1.27)
+				)
+				(hide yes)
+			)
+		)
+		(pin "1"
+		)
+		(instances
+			(project "FLP_PCB_set"
+				(path "/3f8c5218-62bd-4afc-a38b-629e4a961e52/3028588a-b9cc-4609-a7ce-985f9df6b777"
+					(reference "#PWR058")
+					(unit 1)
+				)
+			)
+		)
+	)
+	(symbol
 		(lib_id "Device:C")
 		(at 266.7 48.26 0)
@@
 		(on_board yes)
 		(dnp no)
+		(fields_autoplaced yes)
 		(property "Reference" "C14"
 			(at 104.14 42.164 0)
@@
 			)
 		)
-		(property "Value" "USB_ON"
+		(property "Value" "150080GS75000"
 			(at 180.0225 57.15 0)
 			(effects
@@
 			)
 		)
-		(property "Footprint" "Capacitor_SMD:C_0402_1005Metric"
+		(property "Footprint" "Inductor_SMD:L_0402_1005Metric"
 			(at 256.54 26.67 0)
 			(effects
@@
 			)
 		)
-		(property "Value" "USB_C_Receptacle_USB2.0_16P"
+		(property "Value" "12402012E212A"
 			(at 232.41 118.1099 0)
 			(effects

Commit message: PCB pdf add
Changed lines of the file:
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@@
 	)
 	(junction
-		(at 83.82 170.18)
-		(diameter 0)
-		(color 0 0 0 0)
-	)
-	(junction
 		(at 83.82 91.44)
 		(diameter 0)
@@
 	)
 	(junction
+		(at 83.82 171.45)
+		(diameter 0)
+		(color 0 0 0 0)
+	)
+	(junction
 		(at 259.08 30.48)
 		(diameter 0)
@@
 	(wire
 		(pts
+			(xy 83.82 167.64) (xy 83.82 171.45)
+		)
+		(stroke
+			(width 0)
+			(type default)
+		)
+	)
+	(wire
+		(pts
 			(xy 149.86 78.74) (xy 154.94 78.74)
 		)
@@
 	(wire
 		(pts
-			(xy 83.82 172.72) (xy 83.82 170.18)
+			(xy 83.82 172.72) (xy 83.82 171.45)
 		)
 		(stroke
@@
 	(wire
 		(pts
-			(xy 83.82 167.64) (xy 83.82 170.18)
-		)
-		(stroke
-			(width 0)
-			(type default)
-		)
-	)
-	(wire
-		(pts
 			(xy 29.21 55.88) (xy 33.02 55.88)
 		)
@@
 	(wire
 		(pts
-			(xy 85.09 170.18) (xy 83.82 170.18)
+			(xy 90.17 171.45) (xy 83.82 171.45)
 		)
 		(stroke
@@
 		(on_board yes)
 		(dnp no)
-		(fields_autoplaced yes)
 		(property "Reference" "R1"
-			(at 33.02 163.83 90)
+			(at 27.686 166.878 90)
 			(effects
 				(font
@@
 		)
 		(property "Value" "100R"
-			(at 33.02 166.37 90)
+			(at 27.686 169.418 90)
 			(effects
 				(font
@@
 					(size 1.27 1.27)
 				)
-				(hide yes)
 			)
 		)
@@
 		)
 		(property "Value" "0.1uF"
-			(at 115.824 170.688 90)
+			(at 117.348 170.688 90)
 			(effects
 				(font
@@
 		(dnp no)
 		(property "Reference" "C20"
-			(at 231.1399 71.12 0)
+			(at 231.394 82.042 0)
 			(effects
 				(font
@@
 		)
 		(property "Value" "12pF"
-			(at 233.6799 71.12 0)
+			(at 233.934 82.042 0)
 			(effects
 				(font
@@
 		(on_board yes)
 		(dnp no)
-		(fields_autoplaced yes)
 		(property "Reference" "R2"
-			(at 33.02 166.37 90)
+			(at 39.116 170.18 90)
 			(effects
 				(font
@@
 		)
 		(property "Value" "100R"
-			(at 33.02 168.91 90)
+			(at 39.116 172.72 90)
 			(effects
 				(font
@@
 		(on_board yes)
 		(dnp no)
-		(fields_autoplaced yes)
 		(property "Reference" "C7"
-			(at 76.2 45.7199 0)
+			(at 73.152 49.276 0)
 			(effects
 				(font
@@
 		)
 		(property "Value" "1uF"
-			(at 76.2 48.2599 0)
+			(at 73.152 51.816 0)
 			(effects
 				(font
@@
 	(symbol
 		(lib_id "power:GND")
-		(at 85.09 170.18 90)
+		(at 90.17 171.45 0)
 		(unit 1)
 		(exclude_from_sim no)
@@
 		(fields_autoplaced yes)
 		(property "Reference" "#PWR08"
-			(at 91.44 170.18 0)
+			(at 90.17 177.8 0)
 			(effects
 				(font
@@
 		)
 		(property "Value" "GND"
-			(at 88.9 170.1799 90)
+			(at 92.71 172.7199 0)
 			(effects
 				(font
 					(size 1.27 1.27)
 				)
-				(justify right)
+				(justify left)
 			)
 		)
 		(property "Footprint" ""
-			(at 85.09 170.18 0)
+			(at 90.17 171.45 0)
 			(effects
 				(font
@@
 		)
 		(property "Datasheet" ""
-			(at 85.09 170.18 0)
+			(at 90.17 171.45 0)
 			(effects
 				(font
@@
 		)
 		(property "Description" "Power symbol creates a global label with name \"GND\" , ground"
-			(at 85.09 170.18 0)
+			(at 90.17 171.45 0)
 			(effects
 				(font
@@
 		(on_board yes)
 		(dnp no)
-		(fields_autoplaced yes)
 		(property "Reference" "R4"
-			(at 33.02 171.45 90)
+			(at 38.862 177.038 90)
 			(effects
 				(font
@@
 		)
 		(property "Value" "100R"
-			(at 33.02 173.99 90)
+			(at 38.862 179.578 90)
 			(effects
 				(font
@@
 					(size 1.27 1.27)
 				)
-				(hide yes)
 			)
 		)
@@
 		)
 		(property "Value" "4.7uF"
-			(at 112.522 183.896 90)
+			(at 113.538 183.896 90)
 			(effects
 				(font
@@
 		(on_board yes)
 		(dnp no)
-		(fields_autoplaced yes)
 		(property "Reference" "R7"
-			(at 102.87 44.704 0)
+			(at 101.854 42.926 0)
 			(effects
 				(font
@@
 		)
 		(property "Value" "100K"
-			(at 102.87 42.164 0)
+			(at 103.378 44.45 0)
 			(effects
 				(font
@@
 		(on_board yes)
 		(dnp no)
-		(fields_autoplaced yes)
 		(property "Reference" "R3"
-			(at 33.02 168.91 90)
+			(at 27.178 173.736 90)
 			(effects
 				(font
@@
 		)
 		(property "Value" "100R"
-			(at 33.02 171.45 90)
+			(at 27.178 176.276 90)
 			(effects
 				(font
@@
 		)
 		(property "Value" "5.1K"
-			(at 194.564 124.714 90)
+			(at 194.31 129.286 90)
 			(effects
 				(font
 					(size 1.27 1.27)
 				)
-				(hide yes)
 			)
 		)
@@
 		(dnp no)
 		(property "Reference" "C2"
-			(at 20.574 80.01 0)
+			(at 24.892 81.534 90)
 			(effects
 				(font
@@
 		)
 		(property "Value" "0.1uF"
-			(at 33.02 81.28 0)
+			(at 28.702 84.328 90)
 			(effects
 				(font
@@
 					(size 1.27 1.27)
 				)
-				(hide yes)
 			)
 		)
