File: FLP_device_PCB/FLP_PCB_set/FLP_PCB_set/GPS.kicad_sch (KiCad schematic)
At the start: 3 parts, among them U12 L86-M33

Commit message: PCB pdf add
Changed lines of the file:
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@@
 		(on_board yes)
 		(dnp no)
-		(fields_autoplaced yes)
 		(property "Reference" "C28"
-			(at 100.33 46.9899 0)
+			(at 91.948 46.99 0)
 			(effects
 				(font
@@
 		)
 		(property "Value" "1uF"
-			(at 100.33 49.5299 0)
+			(at 91.948 49.53 0)
 			(effects
 				(font
